Commit message: launch files

File: potato_ws/install/robot_description/share/robot_description/description/inertial_macros.xacro (robot description, xacro)
@@ -1,32 +1 @@
-<?xml version="1.0"?>
-<robot xmlns:xacro="http://www.ros.org/wiki/xacro" >
-    <!-- Specify some standard inertial calculations https://en.wikipedia.org/wiki/List_of_moments_of_inertia -->
-    <!-- These make use of xacro's mathematical functionality -->
-    <xacro:macro name="inertial_sphere" params="mass radius *origin">
-        <inertial>
-            <xacro:insert_block name="origin"/>
-            <mass value="${mass}" />
-            <inertia ixx="${(2/5) * mass * (radius*radius)}" ixy="0.0" ixz="0.0"
-                    iyy="${(2/5) * mass * (radius*radius)}" iyz="0.0"
-                    izz="${(2/5) * mass * (radius*radius)}" />
-        </inertial>
-    </xacro:macro>
-    <xacro:macro name="inertial_box" params="mass x y z *origin">
-        <inertial>
-            <xacro:insert_block name="origin"/>
-            <mass value="${mass}" />
-            <inertia ixx="${(1/12) * mass * (y*y+z*z)}" ixy="0.0" ixz="0.0"
-                    iyy="${(1/12) * mass * (x*x+z*z)}" iyz="0.0"
-                    izz="${(1/12) * mass * (x*x+y*y)}" />
-        </inertial>
-    </xacro:macro>
-    <xacro:macro name="inertial_cylinder" params="mass length radius *origin">
-        <inertial>
-            <xacro:insert_block name="origin"/>
-            <mass value="${mass}" />
-            <inertia ixx="${(1/12) * mass * (3*radius*radius + length*length)}" ixy="0.0" ixz="0.0"
-                    iyy="${(1/12) * mass * (3*radius*radius + length*length)}" iyz="0.0"
-                    izz="${(1/2) * mass * (radius*radius)}" />
-        </inertial>
-    </xacro:macro>
-</robot>
+/home/ws/potato_ws/src/robot_description/description/inertial_macros.xacro

File: potato_ws/install/robot_description/share/robot_description/description/robot.urdf.xacro (robot description, xacro)
@@ -1,4 +1 @@
-<?xml version = "1.0"?>
-<robot xmlns:xacro = "https://www.ros.org/wiki/xacro" name = "demo_bot">
-    <xacro:include filename = "robot_core.xacro"/>
-</robot>
+/home/ws/potato_ws/src/robot_description/description/robot.urdf.xacro

File: potato_ws/install/robot_description/share/robot_description/description/robot_core.xacro (robot description, xacro)
@@ -1,135 +1 @@
-<?xml version="1.0"?>
-<robot xmlns:xacro = "https://www.ros.org/wiki/xacro">
-    <xacro:include filename = "inertial_macros.xacro"/>
-    <!-- MACROS -->
-     <!-- sizes are in meters -->
-     <xacro:property name = "BOX_LENGTH" value = "0.30"/>
-     <xacro:property name = "BOX_HEIGHT" value = "0.15"/>
-     <!-- weight in kg -->
-     <xacro:property name = "BOX_WEIGHT" value = "0.5"/>
-     <xacro:property name = "WHEEL_WEIGHT" value = "0.1"/>
-    <!-- COLORS -->
-    <material name = "white">
-        <color rgba = "1 1 1 1 " />
-    </material>
-    <material name = "black">
-        <color rgba = "0 0 0 1"/>
-    </material>
-    <material name = "purple">
-        <color rgba = "0.227 0 0.871 0.8"/>
-    </material>
-    <material name = "teal">
-        <color rgba = "0.129 0.98 0.98 0.8"/>
-    </material>
-    <!-- BASE LINK -->
-     <!-- setting our base link to be the center of rotation -->
-     <link name = "base_link">
-     </link>
-     <!-- our chassis is going to be a box -->
-      <joint name = "chassis_joint" type = "fixed">
-        <parent link = "base_link"/>
-        <child link = "chassis"/>
-        <!-- origin for this link will be back bottom center, so right behind the base link -->
-        <origin xyz = "-0.1 0 0 "/>
-      </joint>
-    <!-- CHASSIS LINK -->
-      <link name = "chassis">
-        <visual>
-            <!-- moving the origin so the chassis is in the right place -->
-            <origin xyz = "${BOX_LENGTH/2} 0 0.075"/>
-            <geometry>
-                <!-- box size in meters -->
-                <box size = "${BOX_LENGTH} ${BOX_LENGTH} ${BOX_HEIGHT}"/>
-            </geometry>
-            <!-- chassis will be white -->
-            <material name = "white"/>
-        </visual>
-        <!-- COLLISION (just a copy of the viusal but without material) -->
-        <collision>
-            <!-- moving the origin so the chassis is in the right place -->
-            <origin xyz = "${BOX_LENGTH/2} 0 0.075"/>
-            <geometry>
-                <!-- box size in meters -->
-                <box size = "${BOX_LENGTH} ${BOX_LENGTH} ${BOX_HEIGHT}"/>
-            </geometry>
-        </collision>
-        <!-- chassis inertial macros -->
-         <xacro:inertial_box mass = "${BOX_WEIGHT}" x = "${BOX_LENGTH}" y = "${BOX_LENGTH}" z = "${BOX_HEIGHT}">
-            <origin xyz = "0.15 0 0.075" rpy = "0 0 0"/>
-         </xacro:inertial_box>
-      </link>
-    <!-- LEFT WHEEL LINK -->
-    <joint name = "left_wheel_join" type = "continuous">
-        <parent link = "base_link"/>
-        <child link = "left_wheel"/>
-        <!-- rotate wheel along x-axis -->
-        <origin xyz = "0 0.175 0" rpy = "-${pi/2} 0 0"/>
-        <axis xyz = "0 0 1"/>
-    </joint>
-    <link name = "left_wheel">
-        <visual>
-            <geometry>
-                <!-- by default, cylinders in ros are oriented along the z-axis, so we need to rotate along x-axis for wheel -->
-                <cylinder radius = "0.05" length = "0.05"/>
-            </geometry>
-            <material name = "black"/>
-        </visual>
-        <!-- left wheel collision -->
-        <collision>
-            <geometry>
-                <cylinder radius = "0.05" length = "0.05"/>
-            </geometry>
-        </collision>
-        <!-- left wheel inertial macros -->
-         <xacro:inertial_cylinder mass = "${WHEEL_WEIGHT}" length = "0.04" radius = "0.05">
-            <origin xyz = "0 0 0" rpy = "0 0 0"/>
-         </xacro:inertial_cylinder>
-    </link>
-    <!-- RIGHT WHEEL LINK -->
-    <joint name = "right_wheel_join" type = "continuous">
-        <parent link = "base_link"/>
-        <child link = "right_wheel"/>
-        <!-- rotate wheel along x-axis -->
-        <origin xyz = "0 -0.175 0" rpy = "${pi/2} 0 0"/>
-        <axis xyz = "0 0 -1"/>
-    </joint>
-    <link name = "right_wheel">
-        <visual>
-            <geometry>
-                <!-- by default, cylinders in ros are oriented along the z-axis, so we need to rotate along x-axis for wheel -->
-                <cylinder radius = "0.05" length = "0.05"/>
-            </geometry>
-            <material name = "black"/>
-        </visual>
-        <!-- right wheel collision -->
-        <collision>
-            <geometry>
-                <cylinder radius = "0.05" length = "0.05"/>
-            </geometry>
-        </collision>
-        <!-- right wheel inertial macros -->
-         <xacro:inertial_sphere mass = "${WHEEL_WEIGHT}" radius = "0.05">
-            <origin xyz = "0 0 0" rpy = "0 0 0"/>
-         </xacro:inertial_sphere>
-    </link>
-    <!-- CASTER WHEEEL LINK -->
-     <joint name = "caster_wheel_joint" type = "fixed">
-        <parent link = "chassis"/>
-        <child link = "caster_wheel"/>
-        <origin xyz = "0.24 0 0"/>
-     </joint>
-     <link name = "caster_wheel">
-        <visual>
-            <geometry>
-                <sphere radius = "0.05"/>
-            </geometry>
-            <material name = "purple"/>
-        </visual>
-        <!-- COLLISION (just copy visual and change to collision) -->
-         <collision>
-            <geometry>
-                <sphere radius = "0.05"/>
-            </geometry>
-        </collision>
-     </link>
-</robot>
+/home/ws/potato_ws/src/robot_description/description/robot_core.xacro

File: potato_ws/src/robot_description/description/robot.urdf.xacro (robot description, xacro)
@@ -2,3 +2,4 @@
 <robot xmlns:xacro = "https://www.ros.org/wiki/xacro" name = "demo_bot">
     <xacro:include filename = "robot_core.xacro"/>
+    <xacro:include filename = "gazebo_control.xacro"/>
 </robot>

File: potato_ws/src/robot_description/description/robot_core.xacro (robot description, xacro)
@@ -42,6 +42,6 @@
                 <box size = "${BOX_LENGTH} ${BOX_LENGTH} ${BOX_HEIGHT}"/>
             </geometry>
-            <!-- chassis will be white -->
-            <material name = "white"/>
+            <!-- changing the name changes the color of the chassis -->
+            <material name = "purple"/>
         </visual>
         <!-- COLLISION (just a copy of the viusal but without material) -->
