Commit message: gazebo control

File: potato_ws/src/robot_description/description/robot_core.xacro (robot description, xacro)
@@ -43,5 +43,5 @@
             </geometry>
             <!-- changing the name changes the color of the chassis -->
-            <material name = "purple"/>
+            <material name = "white"/>
         </visual>
         <!-- COLLISION (just a copy of the viusal but without material) -->
@@ -59,4 +59,7 @@
          </xacro:inertial_box>
       </link>
+      <gazebo reference = "chassis">
+        <material>Gazebo/White</material>
+      </gazebo>
     <!-- LEFT WHEEL LINK -->
     <joint name = "left_wheel_join" type = "continuous">
@@ -86,4 +89,7 @@
          </xacro:inertial_cylinder>
     </link>
+    <gazebo reference = "left_wheel">
+        <material>Gazebo/Black</material>
+    </gazebo>
     <!-- RIGHT WHEEL LINK -->
     <joint name = "right_wheel_join" type = "continuous">
@@ -113,4 +119,7 @@
          </xacro:inertial_sphere>
     </link>
+    <gazebo reference = "right_wheel">
+        <material>Gazebo/Black</material>
+    </gazebo>
     <!-- CASTER WHEEEL LINK -->
      <joint name = "caster_wheel_joint" type = "fixed">
@@ -132,4 +141,11 @@
             </geometry>
         </collision>
+        <!-- caster wheel inertial macros -->
+        <xacro:inertial_sphere mass = "${WHEEL_WEIGHT}" radius = "0.05">
+            <origin xyz = "0 0 0" rpy = "0 0 0"/>
+        </xacro:inertial_sphere>
      </link>
+    <gazebo reference = "left_wheel">
+        <material>Gazebo/Black</material>
+    </gazebo>
 </robot>
